File: C02.kicad_pcb (KiCad board)
At the start: 2 copper layers, 75.7 x 36.8 mm, 98 parts, among them J1 USB_B_Mini, J10 Conn_01x01, J2 Conn_01x10_Male, J3 Conn_01x06_Male, J4 Conn_01x08_Male, J5 Conn_01x08_Male, J6 Screw_Terminal_01x04, J7 Conn_01x01, J8 Conn_01x01, J9 Conn_01x01, Q1 BC847BS, Q2 BC857BS, Q3 IRLML6344, U1 ATmega328PB-MU, U2 NME0509SC, U3 ISO7742, U4 LM393, U5 MIC5235-5.0, U6 FT230XQ, U7 ISO7742, U8 ISO7740, Y1 16Mhz, 6pF

Commit message: Initial commit
Parts:
- removed C20, C21: 100n, Capacitor_SMD:C_0603_1608Metric
- removed C23: 22p, Capacitor_SMD:C_1206_3216Metric
- removed C3: 47uF/10V, Capacitors_SMD:C_0805
- removed C4: 330n, Capacitor_SMD:C_0603_1608Metric
- removed D7: CDBU0245, Diode_SMD:D_0805_2012Metric
- removed D9: 1N4148W, Diode_SMD:D_MiniMELF
- removed Q1: BC847BS, TO_SOT_Packages_SMD:SOT-363_SC-70-6
- removed Q2: BC857BS, TO_SOT_Packages_SMD:SOT-363_SC-70-6
- removed Q3: IRLML6344, TO_SOT_Packages_SMD:SOT-23
- removed R1: 6.8k, Resistors_SMD:R_0603
- removed R17: 160, Resistor_SMD:R_0805_2012Metric
- removed R18: 100k, Resistors_SMD:R_0603
- removed R2: 22, Resistors_SMD:R_0603
- removed R3: 1k, Resistors_SMD:R_0603
- removed TP1, TP2: TestPoint, TestPoint:TestPoint_Pad_D1.0mm
- removed U5: MIC5235-5.0, TO_SOT_Packages_SMD:SOT-23-5
- added J11: ISP, Connector_PinHeader_2.54mm:PinHeader_2x03_P2.54mm_Vertical, F.Cu at (78.5, 36.4)
- added J12: Conn_01x02, Connector_PinHeader_2.54mm:PinHeader_1x02_P2.54mm_Vertical, F.Cu at (83.6, 36.4)
- added R33: 100k, Resistor_SMD:R_0603_1608Metric, F.Cu at (90.6, 43.7)
- added RN1: 4.7k, Resistor_SMD:R_Array_Concave_4x0603, B.Cu at (92.2, 37.8)
- C1: value 100nF -> 1u/35V
- C10: value 100n -> 1u; footprint Capacitor_SMD:C_1206_3216Metric -> Capacitor_SMD:C_0603_1608Metric; moved to F.Cu
- C12, C13, R21: moved to F.Cu
- C16, C17, C18, C19, C9: value 100n -> 1u
- C2: value 4.7uF/35V -> 10u/25V; footprint Capacitors_SMD:C_0805 -> Capacitor_SMD:C_0603_1608Metric
- C5, C6: footprint Capacitors_SMD:C_0603_HandSoldering -> Capacitor_SMD:C_0603_1608Metric; moved to F.Cu
- C8: value 4.7u/25V -> 10u/25V; moved to F.Cu
- D1: value TX(white) -> D_Schottky; footprint LEDs:LED_0603 -> Diode_SMD:D_0603_1608Metric
- D10: value SSL34 -> SS34FA; footprint Diode_SMD:D_SMC -> Diode_SMD:D_SOD-123F
- D16: value LED -> LED(grn); footprint LEDs:LED_0603 -> LED_SMD:LED_0603_1608Metric
- D19: value SSL34 -> SS34FA; footprint Diode_SMD:D_SMC -> Diode_SMD:D_SOD-123F; moved to B.Cu
- D2: value CDBU0245 -> D_Schottky; footprint Diode_SMD:D_SOD-523 -> Diode_SMD:D_0603_1608Metric
- J1: footprint Frank:USB_Micro-B_Reichelt_BWM_SMD -> RTB:USB_Micro-B_Reichelt_BWM_SMD
- L1: footprint Inductors_SMD:L_0805 -> Inductor_SMD:L_0805_2012Metric; moved to F.Cu
- R10, R12: value 56k -> 100k; footprint Resistors_SMD:R_0603 -> Resistor_SMD:R_0603_1608Metric
- R11, R13, R14, R16, R20, R28, R5, R6, R7, R9: footprint Resistors_SMD:R_0603 -> Resistor_SMD:R_0603_1608Metric
- R15: value 120k -> 100k
- R19, R31, R32: footprint Resistor_SMD:R_0402_1005Metric -> Resistor_SMD:R_0603_1608Metric
- R22, R23: value 10k -> 100k
- R4: value 33k -> 1k; footprint Resistors_SMD:R_0603 -> Resistor_SMD:R_0603_1608Metric
- R8: value 47k -> 1k; footprint Resistors_SMD:R_0603 -> Resistor_SMD:R_0603_1608Metric
- U2: value NME0509SC -> NME0505SC; footprint Frank:DCDC-Conv_muRata_NMAxxxxSC -> RTB:DCDC-Conv_muRata_NMAxxxxSC
- U3: value ISO7742 -> MIC5235-5.0; footprint Housings_SSOP:SSOP-16_3.9x4.9mm_Pitch0.635mm -> Package_TO_SOT_SMD:SOT-23-5
- U6: footprint Housings_DFN_QFN:QFN-16-1EP_4x4mm_Pitch0.65mm -> Package_DFN_QFN:QFN-16-1EP_4x4mm_P0.65mm_EP2.5x2.5mm
- Y1: footprint Crystals:Crystal_SMD_2016-4pin_2.0x1.6mm -> Crystal:Crystal_SMD_2016-4Pin_2.0x1.6mm
- moved C19 15.4 mm to (96.4, 36.4)
- moved U8 15.3 mm to (92.2, 37.8)
- moved D2 14.6 mm to (101.4, 40.3)
- moved C18 14.6 mm to (87.2, 35.7), turned to 180 degrees
- moved R21 14.1 mm to (104.8, 41.3), turned to 90 degrees
- moved U3 13.1 mm to (100.4, 36.9), turned to 90 degrees
- moved C6 12.5 mm to (59.5, 46.0), turned to 90 degrees
- moved D1 11.6 mm to (96.6, 46.7)
- moved D4 10.9 mm to (88.5, 46.5)
- moved D3 10.8 mm to (85.9, 46.5)
- moved L1 10.3 mm to (57.9, 43.3), turned to 90 degrees
- moved R31 10.3 mm to (81.1, 39.2)
- moved R19 9.58 mm to (83.8, 43.7), turned to 270 degrees
- moved C5 8.44 mm to (55.5, 44.3)
- moved C1 7.94 mm to (96.6, 43.7), turned to 90 degrees
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Connections:
- net /RailcomRX/RX+ renamed Net-(R5-Pad2)
- net /Track/bstDCC-2 renamed /Connectors/bstDCC-1
- net RcmPol renamed RCMpol
- C1 pad 2: Net-(C1-Pad2) -> GNDD
- C19 pad 1: /CPU/GNDio -> GNDio
- C19 pad 2: /CPU/VCCio -> Net-(C19-Pad2)
- C2 pad 1: VREG -> GNDio
- C2 pad 2: GNDD -> Net-(C2-Pad2)
- C8 pad 1: Net-(C8-Pad1) -> 5V
- D1 pad 1: RcmTX -> Net-(C1-Pad1)
- D1 pad 2: Net-(D1-Pad2) -> VTRACK
- D2 pad 1: GNDD -> Net-(C2-Pad2)
- D2 pad 2: Net-(C1-Pad1) -> VCCio
- D5 pad 3: RcmRX -> RCMrx
- D8 pad 1: Net-(D8-Pad1) -> GNDS
- D8 pad 2: /USB/VBUS -> Net-(D8-Pad2)
- J1 pad 4: Net-(J1-Pad4) -> (no net)
- J2 pad 1: 5V -> (no net)
- J2 pad 10: /CPU/SS1 -> (no net)
- J2 pad 2: GNDD -> (no net)
- J2 pad 3: ~RESET -> (no net)
- J2 pad 4: /CPU/SCL0 -> (no net)
- J2 pad 5: /CPU/SDA0 -> (no net)
- J2 pad 6: /CPU/SLDalg -> (no net)
- J2 pad 7: /CPU/SCK1 -> (no net)
- J2 pad 8: /CPU/MISO1 -> (no net)
- J2 pad 9: /CPU/MOSI1 -> (no net)
- J3 pad 3: Net-(J3-Pad3) -> (no net)
- J3 pad 4: VTRACK -> (no net)
- J3 pad 5: VREG -> (no net)
- J3 pad 6: Net-(J3-Pad6) -> VTRACK
- J4 pad 1: /CPU/VCCio -> VCCio
- J4 pad 2: /CPU/GNDio -> GNDio
- J4 pad 4: /CPU/xEN -> Net-(J4-Pad4)
- J4 pad 5: /CPU/x2OUT1 -> Net-(J4-Pad5)
- J4 pad 6: /CPU/x2OUT2 -> Net-(J4-Pad6)
- J4 pad 7: /CPU/x2IN1 -> (no net)
- J4 pad 8: /CPU/x2IN2 -> (no net)
- J5 pad 1: /CPU/x1RCMrx -> (no net)
- J5 pad 2: /CPU/x1RCMtx -> (no net)
- J5 pad 3: /CPU/x1PWRpin -> (no net)
- J5 pad 4: /CPU/x1DCCpin -> (no net)
- J5 pad 5: ISPen -> (no net)
- J5 pad 6: TxD -> (no net)
- J5 pad 7: RxD -> (no net)
- J5 pad 8: ~CTS -> (no net)
- R15 pad 1: GNDS -> /USB/VBUS
- R15 pad 2: Net-(D8-Pad1) -> Net-(D8-Pad2)
- R19 pad 2: RcmRX -> RCMrx
- R26 pad 2: ACKpin -> ACK
- R4 pad 1: DCC-1 -> DCC-2
- R4 pad 2: Net-(C1-Pad2) -> Net-(R4-Pad2)
- R6 pad 2: /RailcomRX/RX- -> Net-(R6-Pad2)
- R8 pad 1: /RailcomRX/RX- -> DCC-2
- R8 pad 2: Net-(C1-Pad1) -> Net-(R33-Pad2)
- U1 pad 10: /CPU/OUT1 -> ACK
- U1 pad 19: /CPU/SS1 -> (no net)
- U1 pad 2: ACKpin -> (no net)
- U1 pad 22: /CPU/MOSI1 -> (no net)
- U1 pad 23: /CPU/MISO1 -> (no net)
- U1 pad 24: /CPU/SCK1 -> (no net)
- U1 pad 26: /CPU/SLDalg -> (no net)
- U1 pad 27: /CPU/SDA0 -> (no net)
- U1 pad 28: /CPU/SCL0 -> (no net)
- U1 pad 3: RcmRX -> RCMrx
- U1 pad 30: RcmRX -> RCMrx
- U1 pad 31: RcmTX -> (no net)
- U1 pad 6: /CPU/IN1 -> (no net)
- U1 pad 9: /CPU/OUT2 -> (no net)
- U2 pad 4: Net-(C8-Pad1) -> 5V
- U3 pad 1: 5V -> Net-(C2-Pad2)
- U3 pad 2: GNDD -> GNDio
- U3 pad 3: /CPU/OUT1 -> Net-(C2-Pad2)
- U3 pad 4: /CPU/OUT2 -> (no net)
- U3 pad 5: /CPU/IN1 -> Net-(C19-Pad2)
- U4 pad 2: /RailcomRX/RX- -> Net-(R6-Pad2)
- U4 pad 3: DCC-2 -> Net-(R33-Pad2)
- U4 pad 6: DCC-2 -> Net-(R4-Pad2)
- U4 pad 8: VREG -> Net-(C1-Pad1)
- U6 pad 12: Net-(U6-Pad12) -> (no net)
- U6 pad 14: Net-(U6-Pad14) -> (no net)
- U7 pad 7: VCCIO -> (no net)
- U8 pad 10: /CPU/xEN -> (no net)
- U8 pad 11: /CPU/x1DCCpin -> Net-(RN1-Pad4)
- U8 pad 12: /CPU/x1PWRpin -> Net-(RN1-Pad3)
- U8 pad 13: /CPU/x1RCMtx -> Net-(RN1-Pad2)
- U8 pad 14: /CPU/x1RCMrx -> Net-(RN1-Pad1)
- U8 pad 15: /CPU/GNDio -> GNDio
- U8 pad 16: /CPU/VCCio -> Net-(C19-Pad2)
- U8 pad 3: RcmRX -> DCCpin
- U8 pad 4: RcmTX -> ACK
- U8 pad 5: PWRpin -> RCMrx
- U8 pad 6: DCCpin -> PWRpin
- U8 pad 7: Net-(U8-Pad7) -> (no net)
- U8 pad 9: /CPU/GNDio -> GNDio
- Y1 pad 2: Net-(Y1-Pad2) -> (no net)
- Y1 pad 4: Net-(Y1-Pad4) -> (no net)
Routing:
- net VREG: track 67.2 -> 0.00 mm, vias 1 -> 0
- net RcmTX: track 52.8 -> 0.00 mm, vias 5 -> 0
- net RcmRX: track 48.5 -> 0.00 mm, vias 3 -> 0
- net GNDD: track 76.2 -> 28.2 mm, vias 20 -> 19
- net RCMrx: track 0.00 -> 45.6 mm, vias 0 -> 2
- net ACKpin: track 44.8 -> 0.00 mm, vias 3 -> 0
- net ACK: track 0.00 -> 42.4 mm, vias 0 -> 1
- net VCCIO: track 47.0 -> 10.2 mm, vias 3 -> 4
- net /CPU/xEN: track 35.0 -> 0.00 mm, vias 2 -> 0
- net /CPU/GNDio: track 33.9 -> 0.00 mm, vias 2 -> 0
- net 5V: track 43.4 -> 10.8 mm, vias 8 -> 9
- net /CPU/VCCio: track 28.9 -> 0.00 mm, vias 2 -> 0
- net GNDS: track 47.1 -> 21.9 mm, vias 7 -> 9
- net DCC-1: track 51.9 -> 28.0 mm, vias 3 -> 2
- net GNDio: track 0.00 -> 21.0 mm
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- added copper zone on In2.Cu, net 5V
- added copper zone on In1.Cu, net GNDD
- added copper zone on In1.Cu, net VCCIO
- added copper zone on In2.Cu, net VUSB
- removed copper zone on B.Cu, net 5V
- removed copper zone on F.Cu, net 5V
- removed copper zone on F.Cu, net GNDS
Other:
- copper layers 2 -> 4
- rule pad_to_mask_clearance: 0.2 -> 0
- rule via_min_size: 0.6 -> 0.5
- board text added: "+ - d a r p"
- board text added: "BST"
- board text added: "DCC 1 2"
- board text added: "DPM(C02)"
- board text added: "ISP"
- board text added: "TRK"
- board text added: "fschum'24"
- board text added: "n.c."
- board text removed: "Bot"
- board text removed: "DC/DC"
- board text removed: "DPM (C02)"
- board text removed: "Top"
